Commit message: feat: windranger enable camera

File: windranger/legged_gym/resources/robots/cyberdog2/urdf/cyberdog2.urdf (robot description, URDF)
Before this commit: robot cyberdog2_description, 19 links, 18 joints
Links:
- added link AI_camera_link, mass 0.001; collision box size=.001 .001 .001; visual box size=0.001 0.001 0.001
- added link D435_camera_link, mass 0.001; collision box size=.001 .001 .001; visual box size=0.001 0.001 0.001
- added link RGB_camera_link, mass 0.001; collision box size=.001 .001 .001; visual box size=0.001 0.001 0.001
- added link imu_link, mass 0.001; collision box size=.001 .001 .001; visual box size=0.001 0.001 0.001
- added link lidar_link, mass 0.001
Joints:
- added joint AI_camera_joint: type fixed, parent body, child AI_camera_link, origin xyz=290.228e-3 0 147.420e-3 rpy=0 0 0
- added joint D435_camera_joint: type fixed, parent body, child D435_camera_link, origin xyz=271.994e-3 25e-3 114.912e-3 rpy=0 0 0
- added joint RGB_camera_joint: type fixed, parent body, child RGB_camera_link, origin xyz=275.76e-3 0 125.794e-3 rpy=0 0 0
- added joint imu_joint: type fixed, parent body, child imu_link, origin xyz=33.4e-3 -17.2765e-3 51.0469e-3 rpy=0 0 0
- added joint scan_joint: type fixed, parent body, child lidar_link, origin xyz=0.21425 0 0.0908 rpy=0 0 0

File: windranger/legged_gym/resources/robots/cyberdog2/xacro/robot.xacro (robot description, xacro)
@@ -65,5 +65,5 @@
         </inertial>
     </link>
-    <!-- <joint name="imu_joint" type="fixed">
+    <joint name="imu_joint" type="fixed">
         <parent link="body" />
         <child link="imu_link" />
@@ -172,5 +172,5 @@
             </geometry>
         </collision>
-    </link> -->
+    </link>
     <xacro:leg name="FR" mirror="-1" mirror_dae="False" front_hind="1" front_hind_dae="True">
         <origin rpy="0 0 0" xyz="${abad_offset_x} ${-abad_offset_y} 0" />
