Commit message: fix: fix play script module not found and change the link name of urdf.

File: assets/cyberdog_robot/cyberdog2.urdf (robot description, URDF)
Before this commit: robot cyber_dog, 40 links, 39 joints
Links:
- removed link FL_abad
- removed link FL_abad_rotor
- removed link FL_hip_shoulder
- removed link FL_knee
- removed link FL_knee_rotor
- removed link FR_abad
- removed link FR_abad_rotor
- removed link FR_hip_shoulder
- removed link FR_knee
- removed link FR_knee_rotor
- removed link RL_abad
- removed link RL_abad_rotor
- removed link RL_hip_shoulder
- removed link RL_knee
- removed link RL_knee_rotor
- removed link RR_abad
- removed link RR_abad_rotor
- removed link RR_hip_shoulder
- removed link RR_knee
- removed link RR_knee_rotor
- removed link base_link
- added link FL_calf, mass 0.116; collision box size=0.016 0.016 0.18341; collision sphere radius=0.016
- added link FL_calf_rotor, mass 0.0567
- added link FL_thigh, mass 0.482; collision box size=0.12 0.025 0.034; visual mesh filename=file://./cyberdog_description/meshes/hip.dae scale=1 1 1
- added link FL_thigh_rotor, mass 0.0567
- added link FL_thigh_shoulder; collision cylinder length=0.035 radius=0.039
- added link FR_calf, mass 0.116; collision box size=0.016 0.016 0.18341; collision sphere radius=0.016
- added link FR_calf_rotor, mass 0.0567
- added link FR_thigh, mass 0.482; collision box size=0.12 0.025 0.034; visual mesh filename=file://./cyberdog_description/meshes/hip_mirror.dae scale=1 1 1
- added link FR_thigh_rotor, mass 0.0567
- added link FR_thigh_shoulder; collision cylinder length=0.035 radius=0.039
- added link RL_calf, mass 0.116; collision box size=0.016 0.016 0.18341; collision sphere radius=0.016
- added link RL_calf_rotor, mass 0.0567
- added link RL_thigh, mass 0.482; collision box size=0.12 0.025 0.034; visual mesh filename=file://./cyberdog_description/meshes/hip.dae scale=1 1 1
- added link RL_thigh_rotor, mass 0.0567
- added link RL_thigh_shoulder; collision cylinder length=0.035 radius=0.039
- added link RR_calf, mass 0.116; collision box size=0.016 0.016 0.18341; collision sphere radius=0.016
- added link RR_calf_rotor, mass 0.0567
- added link RR_thigh, mass 0.482; collision box size=0.12 0.025 0.034; visual mesh filename=file://./cyberdog_description/meshes/hip_mirror.dae scale=1 1 1
- added link RR_thigh_rotor, mass 0.0567
- added link RR_thigh_shoulder; collision cylinder length=0.035 radius=0.039
- link FL_hip: mass 0.482 -> 0.354; geometry collision cylinder length=0.035 radius=0.039; visual mesh filename=file://./cyberdog_description/meshes/abad.dae scale=1 1 1
- link FR_hip: mass 0.482 -> 0.354; geometry collision cylinder length=0.035 radius=0.039; visual mesh filename=file://./cyberdog_description/meshes/abad.dae scale=1 1 1
- link RL_hip: mass 0.482 -> 0.354; geometry collision cylinder length=0.035 radius=0.039; visual mesh filename=file://./cyberdog_description/meshes/abad.dae scale=1 1 1
- link RR_hip: mass 0.482 -> 0.354; geometry collision cylinder length=0.035 radius=0.039; visual mesh filename=file://./cyberdog_description/meshes/abad.dae scale=1 1 1
- link base: geometry collision box size=0.236 0.19 0.109; visual mesh filename=file://./cyberdog_description/meshes/body.dae scale=1 1 1
Joints:
- removed joint FL_abad_fixed
- removed joint FL_abad_joint
- removed joint FL_abad_rotor_fix
- removed joint FL_knee_joint
- removed joint FL_knee_rotor_fix
- removed joint FR_abad_fixed
- removed joint FR_abad_joint
- removed joint FR_abad_rotor_fix
- removed joint FR_knee_joint
- removed joint FR_knee_rotor_fix
- removed joint RL_abad_fixed
- removed joint RL_abad_joint
- removed joint RL_abad_rotor_fix
- removed joint RL_knee_joint
- removed joint RL_knee_rotor_fix
- removed joint RR_abad_fixed
- removed joint RR_abad_joint
- removed joint RR_abad_rotor_fix
- removed joint RR_knee_joint
- removed joint RR_knee_rotor_fix
- removed joint floating_base
- added joint FL_calf_joint: type revolute, parent FL_thigh, child FL_calf, origin xyz=0 0 -0.12 rpy=0 0 0, axis 0 1 0, limit lower=-2.5307274153917776 upper=-0.5235987755982988 effort=12.0001 velocity=30.9971
- added joint FL_calf_rotor_fix: type fixed, parent FL_thigh, child FL_calf_rotor, origin xyz=0 -0.0342303 0 rpy=0 0 0
- added joint FL_hip_fixed: type fixed, parent FL_hip, child FL_thigh_shoulder, origin xyz=0 0.059 0 rpy=0 0 0
- added joint FL_thigh_joint: type revolute, parent FL_hip, child FL_thigh, origin xyz=0 0.094 0 rpy=0 0 0, axis 0 1 0, limit lower=-1.3264502315156903 upper=2.792526803190927 effort=12.0001 velocity=30.9971
- added joint FL_thigh_rotor_fix: type fixed, parent FL_thigh, child FL_thigh_rotor, origin xyz=0 -0.07577 0 rpy=0 0 0
- added joint FR_calf_joint: type revolute, parent FR_thigh, child FR_calf, origin xyz=0 0 -0.12 rpy=0 0 0, axis 0 1 0, limit lower=-2.5307274153917776 upper=-0.5235987755982988 effort=12.0001 velocity=30.9971
- added joint FR_calf_rotor_fix: type fixed, parent FR_thigh, child FR_calf_rotor, origin xyz=0 0.0342303 0 rpy=0 0 0
- added joint FR_hip_fixed: type fixed, parent FR_hip, child FR_thigh_shoulder, origin xyz=0 -0.059 0 rpy=0 0 0
- added joint FR_thigh_joint: type revolute, parent FR_hip, child FR_thigh, origin xyz=0 -0.094 0 rpy=0 0 0, axis 0 1 0, limit lower=-1.3264502315156903 upper=2.792526803190927 effort=12.0001 velocity=30.9971
- added joint FR_thigh_rotor_fix: type fixed, parent FR_thigh, child FR_thigh_rotor, origin xyz=0 0.07577 0 rpy=0 0 0
- added joint RL_calf_joint: type revolute, parent RL_thigh, child RL_calf, origin xyz=0 0 -0.12 rpy=0 0 0, axis 0 1 0, limit lower=-2.5307274153917776 upper=-0.5235987755982988 effort=12.0001 velocity=30.9971
- added joint RL_calf_rotor_fix: type fixed, parent RL_thigh, child RL_calf_rotor, origin xyz=0 -0.0342303 0 rpy=0 0 0
- added joint RL_hip_fixed: type fixed, parent RL_hip, child RL_thigh_shoulder, origin xyz=0 0.059 0 rpy=0 0 0
- added joint RL_thigh_joint: type revolute, parent RL_hip, child RL_thigh, origin xyz=0 0.094 0 rpy=0 0 0, axis 0 1 0, limit lower=-0.9773843811168246 upper=3.141592653589793 effort=12.0001 velocity=30.9971
- added joint RL_thigh_rotor_fix: type fixed, parent RL_thigh, child RL_thigh_rotor, origin xyz=0 -0.07577 0 rpy=0 0 0
- added joint RR_calf_joint: type revolute, parent RR_thigh, child RR_calf, origin xyz=0 0 -0.12 rpy=0 0 0, axis 0 1 0, limit lower=-2.5307274153917776 upper=-0.5235987755982988 effort=12.0001 velocity=30.9971
- added joint RR_calf_rotor_fix: type fixed, parent RR_thigh, child RR_calf_rotor, origin xyz=0 0.0342303 0 rpy=0 0 0
- added joint RR_hip_fixed: type fixed, parent RR_hip, child RR_thigh_shoulder, origin xyz=0 -0.059 0 rpy=0 0 0
- added joint RR_thigh_joint: type revolute, parent RR_hip, child RR_thigh, origin xyz=0 -0.094 0 rpy=0 0 0, axis 0 1 0, limit lower=-0.9773843811168246 upper=3.141592653589793 effort=12.0001 velocity=30.9971
- added joint RR_thigh_rotor_fix: type fixed, parent RR_thigh, child RR_thigh_rotor, origin xyz=0 0.07577 0 rpy=0 0 0
- joint FL_foot_fixed: parent FL_knee -> FL_calf
- joint FL_hip_joint: axis 0 1 0 -> 1 0 0; limit lower=-1.3264502315156903 upper=2.792526803190927 effort=12.0001 velocity=30.9971 -> lower=-0.6806784082777885 upper=0.6806784082777885 effort=12.0001 velocity=30.9971; origin xyz=0 0.094 0 rpy=0 0 0 -> xyz=0.164 0.042 0 rpy=0 0 0; parent FL_abad -> base
- joint FL_hip_rotor_fix: origin xyz=0 -0.07577 0 rpy=0 0 0 -> xyz=-0.0642303 0 0 rpy=0 0 0
- joint FR_foot_fixed: parent FR_knee -> FR_calf
- joint FR_hip_joint: axis 0 1 0 -> 1 0 0; limit lower=-1.3264502315156903 upper=2.792526803190927 effort=12.0001 velocity=30.9971 -> lower=-0.6806784082777885 upper=0.6806784082777885 effort=12.0001 velocity=30.9971; origin xyz=0 -0.094 0 rpy=0 0 0 -> xyz=0.164 -0.042 0 rpy=0 0 0; parent FR_abad -> base
- joint FR_hip_rotor_fix: origin xyz=0 0.07577 0 rpy=0 0 0 -> xyz=-0.0642303 0 0 rpy=0 0 0
- joint RL_foot_fixed: parent RL_knee -> RL_calf
- joint RL_hip_joint: axis 0 1 0 -> 1 0 0; limit lower=-0.9773843811168246 upper=3.141592653589793 effort=12.0001 velocity=30.9971 -> lower=-0.6806784082777885 upper=0.6806784082777885 effort=12.0001 velocity=30.9971; origin xyz=0 0.094 0 rpy=0 0 0 -> xyz=-0.164 0.042 0 rpy=0 0 0; parent RL_abad -> base
- joint RL_hip_rotor_fix: origin xyz=0 -0.07577 0 rpy=0 0 0 -> xyz=0.0642303 0 0 rpy=0 0 0
- joint RR_foot_fixed: parent RR_knee -> RR_calf
- joint RR_hip_joint: axis 0 1 0 -> 1 0 0; limit lower=-0.9773843811168246 upper=3.141592653589793 effort=12.0001 velocity=30.9971 -> lower=-0.6806784082777885 upper=0.6806784082777885 effort=12.0001 velocity=30.9971; origin xyz=0 -0.094 0 rpy=0 0 0 -> xyz=-0.164 -0.042 0 rpy=0 0 0; parent RR_abad -> base
- joint RR_hip_rotor_fix: origin xyz=0 0.07577 0 rpy=0 0 0 -> xyz=0.0642303 0 0 rpy=0 0 0
